File: hardware/Wheels Board/Wheels Board.kicad_pcb (KiCad board)
At the start: 2 copper layers, 92.9 x 69.7 mm, 46 parts, among them J1 Conn_01x05, J10 gnd, J11 hall_out, J12 Conn_01x05, J2 24v, J3 Conn_01x03, J4 53307-2471, J6 Conn_01x05_Pin, J7 Conn_01x07, J8 24v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

Commit message: remove old prod files
Routing:
- net /IMU_INT2: track 44.8 -> 43.2 mm
Other:
- board text removed: "unconnected gpio on esp"
Changed lines of the file:
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@@
 		)
 	)
-	(gr_text "unconnected gpio on esp"
-		(at 156.1 74.4 0)
-		(layer "F.SilkS")
-		(effects
-			(font
-				(size 1 1)
-				(thickness 0.15)
-			)
-		)
-	)
 	(gr_text "Wheels board Rev B <3"
 		(at 92.8 81.3 0)
@@
 	)
 	(segment
-		(start 113.321828 96.2)
-		(end 113.35 96.2)
-		(width 0.2)
-		(layer "F.Cu")
-		(net 2)
-	)
-	(segment
 		(start 113.812369 89.569185)
 		(end 113.568673 89.569185)
@@
 	)
 	(segment
-		(start 111.2 96.1)
-		(end 111.9 96.8)
-		(width 0.2)
-		(layer "F.Cu")
-		(net 32)
-	)
-	(segment
 		(start 111.887499 93.1103)
 		(end 111.887499 94.4375)
@@
 	)
 	(segment
-		(start 107.6 95.6)
-		(end 101.35 101.85)
+		(start 127.001 102.101)
+		(end 128.089601 103.189601)
 		(width 0.2)
 		(layer "F.Cu")
@@
 	)
 	(segment
-		(start 111.9 96.8)
-		(end 116.0329 96.8)
+		(start 107.6 95.6)
+		(end 101.35 101.85)
 		(width 0.2)
 		(layer "F.Cu")
@@
 	)
 	(segment
-		(start 127.001 102.101)
-		(end 121.3339 102.101)
+		(start 128.089601 103.189601)
+		(end 128.089601 104.37)
 		(width 0.2)
 		(layer "F.Cu")
@@
 	)
 	(segment
-		(start 96.4 103.8)
-		(end 95.689999 103.8)
+		(start 113.224999 96.1)
+		(end 115.3329 96.1)
 		(width 0.2)
 		(layer "F.Cu")
@@
 	)
 	(segment
-		(start 111.887499 94.4375)
-		(end 111.724999 94.6)
+		(start 96.4 103.8)
+		(end 95.689999 103.8)
 		(width 0.2)
 		(layer "F.Cu")
@@
 	)
 	(segment
-		(start 111.2 95.124999)
-		(end 111.2 96.1)
+		(start 111.887499 94.4375)
+		(end 111.724999 94.6)
 		(width 0.2)
 		(layer "F.Cu")
@@
 	(segment
 		(start 111.724999 94.6)
-		(end 110.724999 95.6)
-		(width 0.2)
-		(layer "F.Cu")
-		(net 32)
-	)
-	(segment
-		(start 98.4 101.85)
-		(end 96.45 103.8)
+		(end 113.224999 96.1)
 		(width 0.2)
 		(layer "F.Cu")
@@
 	)
 	(segment
-		(start 128.089601 104.37)
-		(end 128.089601 103.189601)
+		(start 121.3339 102.101)
+		(end 127.001 102.101)
 		(width 0.2)
 		(layer "F.Cu")
@@
 	)
 	(segment
-		(start 128.089601 103.189601)
-		(end 127.001 102.101)
+		(start 111.724999 94.6)
+		(end 110.724999 95.6)
 		(width 0.2)
 		(layer "F.Cu")
@@
 	)
 	(segment
-		(start 111.2 95.124999)
-		(end 111.724999 94.6)
+		(start 98.4 101.85)
+		(end 96.45 103.8)
 		(width 0.2)
 		(layer "F.Cu")
@@
 	)
 	(segment
-		(start 121.3339 102.101)
-		(end 116.0329 96.8)
+		(start 115.3329 96.1)
+		(end 121.3339 102.101)
 		(width 0.2)
 		(layer "F.Cu")
@@
 	)
 	(zone
-		(net 5)
-		(net_name "Net-(U4-COMP)")
+		(net 45)
+		(net_name "/24v to 5v convertor/ROSC")
 		(layer "F.Cu")
 		(name "$teardrop_padvia$")
 		(hatch none 0.1)
-		(priority 30009)
+		(priority 30011)
 		(attr
 			(teardrop
@@
 		(polygon
 			(pts
-				(xy 80.318968 88.890414) (xy 79.965415 89.243967) (xy 80.090001 90.103013) (xy 80.415708 90.061707)
-				(xy 80.542462 89.297)
+				(xy 80.665001 83.55) (xy 80.165001 83.55) (xy 80.090001 83.875) (xy 80.415001 84.64) (xy 80.740001 83.875)
 			)
 		)
 	)
 	(zone
-		(net 6)
-		(net_name "Net-(C8-Pad2)")
+		(net 5)
+		(net_name "Net-(U4-COMP)")
 		(layer "F.Cu")
 		(name "$teardrop_padvia$")
 		(hatch none 0.1)
-		(priority 30003)
+		(priority 30000)
 		(attr
 			(teardrop
@@
 		(polygon
 			(pts
-				(xy 76.8896 88.0598) (xy 76.8896 87.5598) (xy 76.267987 87.362778) (xy 75.9386 87.832199) (xy 76.271163 88.299497)
+				(xy 78.432124 88.945231) (xy 78.078571 88.591678) (xy 77.354748 88.997302) (xy 77.488293 89.535509)
+				(xy 77.964 89.731553)
 			)
 		)
 	)
 	(zone
-		(net 8)
-		(net_name "/24v to 5v convertor/IND_NODE")
+		(net 6)
+		(net_name "Net-(C8-Pad2)")
 		(layer "F.Cu")
-		(hatch edge 0.5)
-		(priority 4)
+		(name "$teardrop_padvia$")
+		(hatch none 0.1)
+		(priority 30008)
+		(attr
+			(teardrop
+				(type padvia)
+			)
+		)
 		(connect_pads yes
-			(clearance 0.1)
+			(clearance 0)
 		)
-		(min_thickness 0.25)
+		(min_thickness 0.0254)
 		(filled_areas_thickness no)
 		(fill yes
 			(thermal_gap 0.5)
 			(thermal_bridge_width 0.5)
+			(island_removal_mode 1)
+			(island_area_min 10)
 		)
 		(polygon
 			(pts
-				(xy 82.350917 88.939309) (xy 87.25 89.6) (xy 89.1 95.8) (xy 89 100.6) (xy 84 100.5) (xy 82.2 90.7)
+				(xy 76.539 87.5598) (xy 76.539 88.0598) (xy 77.094131 88.2848) (xy 77.49 87.8098) (xy 77.094131 87.3348)
 			)
 		)
 	)
 	(zone
-		(net 3)
-		(net_name "+24V")
+		(net 5)
+		(net_name "Net-(U4-COMP)")
 		(layer "F.Cu")
 		(name "$teardrop_padvia$")
 		(hatch none 0.1)
-		(priority 30007)
+		(priority 30009)
 		(attr
 			(teardrop
@@
 		(polygon
 			(pts
-				(xy 82.75 83.0625) (xy 82.75 82.5625) (xy 82.194869 82.3375) (xy 81.799 82.8125) (xy 82.194869 83.2875)
+				(xy 80.318968 88.890414) (xy 79.965415 89.243967) (xy 80.090001 90.103013) (xy 80.415708 90.061707)
+				(xy 80.542462 89.297)
 			)
 		)
 	)
 	(zone
-		(net 5)
-		(net_name "Net-(U4-COMP)")
+		(net 3)
+		(net_name "+24V")
 		(layer "F.Cu")
 		(name "$teardrop_padvia$")
 		(hatch none 0.1)
-		(priority 30000)
+		(priority 30010)
 		(attr
 			(teardrop
@@
 		(polygon
 			(pts
-				(xy 78.432124 88.945231) (xy 78.078571 88.591678) (xy 77.354748 88.997302) (xy 77.488293 89.535509)
-				(xy 77.964 89.731553)
+				(xy 81.935001 83.55) (xy 81.435001 83.55) (xy 81.360001 83.875) (xy 81.685001 84.64) (xy 82.010001 83.875)
 			)
 		)
@@
 	)
 	(zone
-		(net 7)
-		(net_name "Net-(U4-BOOT)")
+		(net 6)
+		(net_name "Net-(C8-Pad2)")
 		(layer "F.Cu")
 		(name "$teardrop_padvia$")
 		(hatch none 0.1)
-		(priority 30002)
+		(priority 30003)
 		(attr
 			(teardrop
@@
 		(polygon
 			(pts
-				(xy 84.85 87.412498) (xy 84.35 87.412498) (xy 84.143079 88.034111) (xy 84.6 88.425998) (xy 85.056921 88.034111)
+				(xy 76.8896 88.0598) (xy 76.8896 87.5598) (xy 76.267987 87.362778) (xy 75.9386 87.832199) (xy 76.271163 88.299497)
 			)
 		)
 	)
 	(zone
-		(net 9)
-		(net_name "+5V")
+		(net 8)
+		(net_name "/24v to 5v convertor/IND_NODE")
 		(layer "F.Cu")
 		(hatch edge 0.5)
@@
 			(clearance 0.1)
 		)
-		(min_thickness 0.1)
+		(min_thickness 0.25)
 		(filled_areas_thickness no)
 		(fill yes
-			(thermal_gap 0.1)
+			(thermal_gap 0.5)
 			(thermal_bridge_width 0.5)
 		)
 		(polygon
 			(pts
-				(xy 78.639835 89.05) (xy 79.695 89.05) (xy 80.3 95.1) (xy 80.25 100.55) (xy 75.843032 100.5) (xy 74.293032 98.75)
-				(xy 74.143032 94.7) (xy 78.15 93.8)
+				(xy 82.350917 88.939309) (xy 87.25 89.6) (xy 89.1 95.8) (xy 89 100.6) (xy 84 100.5) (xy 82.2 90.7)
 			)
 		)
 	)
 	(zone
-		(net 45)
-		(net_name "/24v to 5v convertor/ROSC")
+		(net 3)
+		(net_name "+24V")
 		(layer "F.Cu")
 		(name "$teardrop_padvia$")
 		(hatch none 0.1)
-		(priority 30004)
+		(priority 30007)
 		(attr
 			(teardrop
@@
 		(polygon
 			(pts
-				(xy 80.165001 83.824999) (xy 80.665001 83.824999) (xy 80.725002 83.112499) (xy 80.250002 82.861499)
-				(xy 79.838198 83.27091)
+				(xy 82.75 83.0625) (xy 82.75 82.5625) (xy 82.194869 82.3375) (xy 81.799 82.8125) (xy 82.194869 83.2875)
 			)
 		)
 	)
 	(zone
-		(net 45)
-		(net_name "/24v to 5v convertor/ROSC")
+		(net 3)
+		(net_name "+24V")
 		(layer "F.Cu")
 		(name "$teardrop_padvia$")
 		(hatch none 0.1)
-		(priority 30011)
+		(priority 30006)
 		(attr
 			(teardrop
@@
 		(polygon
 			(pts
-				(xy 80.665001 83.55) (xy 80.165001 83.55) (xy 80.090001 83.875) (xy 80.415001 84.64) (xy 80.740001 83.875)
+				(xy 82.45 82.5625) (xy 82.45 83.0625) (xy 83.005131 83.2875) (xy 83.401 82.8125) (xy 83.005131 82.3375)
 			)
 		)
 	)
 	(zone
-		(net 3)
-		(net_name "+24V")
+		(net 9)
+		(net_name "+5V")
 		(layer "F.Cu")
-		(name "$teardrop_padvia$")
-		(hatch none 0.1)
-		(priority 30010)
-		(attr
-			(teardrop
-				(type padvia)
-			)
-		)
+		(hatch edge 0.5)
+		(priority 4)
 		(connect_pads yes
-			(clearance 0)
+			(clearance 0.1)
 		)
-		(min_thickness 0.0254)
+		(min_thickness 0.1)
 		(filled_areas_thickness no)
 		(fill yes
-			(thermal_gap 0.5)
+			(thermal_gap 0.1)
 			(thermal_bridge_width 0.5)
-			(island_removal_mode 1)
-			(island_area_min 10)
 		)
 		(polygon
 			(pts
-				(xy 81.935001 83.55) (xy 81.435001 83.55) (xy 81.360001 83.875) (xy 81.685001 84.64) (xy 82.010001 83.875)
+				(xy 78.639835 89.05) (xy 79.695 89.05) (xy 80.3 95.1) (xy 80.25 100.55) (xy 75.843032 100.5) (xy 74.293032 98.75)
+				(xy 74.143032 94.7) (xy 78.15 93.8)
 			)
 		)
 	)
 	(zone
-		(net 3)
-		(net_name "+24V")
+		(net 45)
+		(net_name "/24v to 5v convertor/ROSC")
 		(layer "F.Cu")
 		(name "$teardrop_padvia$")
 		(hatch none 0.1)
-		(priority 30005)
+		(priority 30004)
 		(attr
 			(teardrop
@@
 		(polygon
 			(pts
-				(xy 84.35 83.0625) (xy 84.35 82.5625) (xy 83.794869 82.3375) (xy 83.399 82.8125) (xy 83.794869 83.2875)
+				(xy 80.165001 83.824999) (xy 80.665001 83.824999) (xy 80.725002 83.112499) (xy 80.250002 82.861499)
+				(xy 79.838198 83.27091)
 			)
 		)
 	)
 	(zone
-		(net 6)
-		(net_name "Net-(C8-Pad2)")
+		(net 7)
+		(net_name "Net-(U4-BOOT)")
 		(layer "F.Cu")
 		(name "$teardrop_padvia$")
 		(hatch none 0.1)
-		(priority 30008)
+		(priority 30002)
 		(attr
 			(teardrop
@@
 		(polygon
 			(pts
-				(xy 76.539 87.5598) (xy 76.539 88.0598) (xy 77.094131 88.2848) (xy 77.49 87.8098) (xy 77.094131 87.3348)
+				(xy 84.85 87.412498) (xy 84.35 87.412498) (xy 84.143079 88.034111) (xy 84.6 88.425998) (xy 85.056921 88.034111)
 			)
 		)
@@
 		(name "$teardrop_padvia$")
 		(hatch none 0.1)
-		(priority 30006)
+		(priority 30005)
 		(attr
 			(teardrop
@@
 		(polygon
 			(pts
-				(xy 82.45 82.5625) (xy 82.45 83.0625) (xy 83.005131 83.2875) (xy 83.401 82.8125) (xy 83.005131 82.3375)
+				(xy 84.35 83.0625) (xy 84.35 82.5625) (xy 83.794869 82.3375) (xy 83.399 82.8125) (xy 83.794869 83.2875)
 			)
 		)
