File: hardware/MCU+USB.kicad_sch (KiCad schematic)
At the start: 0 parts

Commit message: Please Final Review
Parts:
- added D13, D15, D16: LED, LED_SMD:LED_0603_1608Metric_Pad1.05x0.95mm_HandSolder, symbol lhrs_misc:Blue_LED
- added R27, R28, R34: 1k, Package_SO:SOIC-14_3.9x8.7mm_P1.27mm, symbol Device:R
Connections:
- net 48PinMCU/PB11: now also R34.1
- net 48PinMCU/PB13: now also R27.1
- net 48PinMCU/PB15: now also R28.1
- net GND: now also D13.1 (K), D15.1 (K), D16.1 (K)
- new net: D13.2 (A), R27.2
- new net: D15.2 (A), R28.2
- new net: D16.2 (A), R34.2
- no-connect marks 2 -> 15

Commit message: Changed MAG to SPI
Connections:
- no-connect marks 15 -> 16
