File: hardware/PowerProtection.kicad_sch (KiCad schematic)
At the start: 18 parts, among them IC2 LM74502DDFR, Q1 PSMN012-100YS, Q2 PSMN012-100YS

Commit message: Updated KiCAD Sharepoint
Parts:
- C29, C34, C35: value 0.1uF -> 0.1u
- C30: value 1uF -> 1u
- C31: value 220nF -> 220n
- C32: value 10uF -> 10n
- C33: value 10uF -> 10u; footprint Capacitor_SMD:C_0603_1608Metric_Pad1.08x0.95mm_HandSolder -> Capacitor_SMD:C_0805_2012Metric_Pad1.18x1.45mm_HandSolder
- IC2: Manufacturer_Name Texas Instruments -> (none); Manufacturer_Part_Number LM74502DDFR -> (none); Mouser Part Number 595-LM74502DDFR -> (none); Mouser Price/Stock https://www.mouser.co.uk/ProductDetail/Texas-Instruments/LM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 -> (none)
- R15, R17, R18, R19, R20: symbol Device:R_US -> Device:R
- R16: symbol Device:R_US -> Device:R; Mouser Part Number 594-MCT06030C3309FP5 -> (none)
- renumbered D9 to D7, D10 to D8
Other:
- note added: "Supp Battery Range: 10V-14.7V"
