File: hardware/power_Rail.kicad_sch (KiCad schematic)
At the start: 18 parts

Commit message: Please Final Review
Changed lines of the file:
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@@
 	(text "Galvanically Isolated"
 		(exclude_from_sim no)
-		(at 187.706 74.676 0)
+		(at 187.96 74.93 0)
 		(effects
 			(font

Commit message: Ready for Final Schematic Review
Changed lines of the file:
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@@
 	(text "Galvanically Isolated"
 		(exclude_from_sim no)
-		(at 187.96 74.93 0)
+		(at 187.198 74.93 0)
 		(effects
 			(font

Commit message: Changed MAG to SPI
Parts:
- removed TP6: 12V_Point, LHRS_Connectors:Molex_Nano-Fit_105310-xx10_2x05_P2.50mm_Vertical, symbol Connector:TestPoint
Connections:
- net MUX_OUT renamed LDO/Vin
Other:
- note removed: "Galvanically Isolated"
Changed lines of the file:
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@@
-		)
-	)
-	(text "Galvanically Isolated"
-		(exclude_from_sim no)
-		(at 187.198 74.93 0)
-		(effects
-			(font
-				(size 1.27 1.27)
-			)
 		)
 	)
@@
 	)
 	(junction
-		(at 109.22 69.85)
-		(diameter 0)
-		(color 0 0 0 0)
-	)
-	(junction
 		(at 109.22 81.28)
 		(diameter 0)
@@
 	(wire
 		(pts
-			(xy 181.61 81.28) (xy 186.69 81.28)
+			(xy 181.61 81.28) (xy 198.12 81.28)
 		)
 		(stroke
@@
 	(wire
 		(pts
-			(xy 189.23 81.28) (xy 198.12 81.28)
-		)
-		(stroke
-			(width 0)
-			(type default)
-		)
-	)
-	(wire
-		(pts
 			(xy 218.44 81.28) (xy 222.25 81.28)
 		)
@@
 		)
 	)
-	(polyline
-		(pts
-			(xy 187.96 76.2) (xy 187.96 88.9)
-		)
-		(stroke
-			(width 0)
-			(type default)
-		)
-	)
 	(wire
 		(pts
@@
 			(width 0)
 			(type default)
-		)
-	)
-	(label "MUX_OUT"
-		(at 189.23 81.28 0)
-		(effects
-			(font
-				(size 1.27 1.27)
-			)
-			(justify left bottom)
 		)
 	)
@@
 			)
 			(justify left bottom)
-		)
-	)
-	(label "MUX_OUT"
-		(at 186.69 81.28 180)
-		(effects
-			(font
-				(size 1.27 1.27)
-			)
-			(justify right bottom)
 		)
 	)
@@
 					(unit 1)
 				)
-			)
-		)
-	)
-	(symbol
-		(lib_id "Connector:TestPoint")
-		(at 109.22 69.85 270)
-		(unit 1)
-		(body_style 1)
-		(exclude_from_sim no)
-		(in_bom yes)
-		(on_board yes)
-		(in_pos_files yes)
-		(dnp no)
-		(fields_autoplaced yes)
-		(property "Reference" "TP6"
-			(at 114.3 68.5799 90)
-			(show_name no)
-			(do_not_autoplace no)
-			(effects
-				(font
-					(size 1.27 1.27)
-				)
-				(justify left)
-			)
-		)
-		(property "Value" "12V_Point"
-			(at 114.3 71.1199 90)
-			(show_name no)
-			(do_not_autoplace no)
-			(effects
-				(font
-					(size 1.27 1.27)
-				)
-				(justify left)
-			)
-		)
-		(property "Footprint" "LHRS_Connectors:Molex_Nano-Fit_105310-xx10_2x05_P2.50mm_Vertical"
-			(at 109.22 74.93 0)
-			(hide yes)
-			(show_name no)
-			(do_not_autoplace no)
-			(effects
-				(font
-					(size 1.27 1.27)
-				)
-			)
-		)
-		(property "Datasheet" ""
-			(at 109.22 74.93 0)
-			(hide yes)
-			(show_name no)
-			(do_not_autoplace no)
-			(effects
-				(font
-					(size 1.27 1.27)
-				)
-			)
-		)
-		(property "Description" "test point"
-			(at 109.22 69.85 0)
-			(hide yes)
-			(show_name no)
-			(do_not_autoplace no)
-			(effects
-				(font
-					(size 1.27 1.27)
-				)
-			)
-		)
-		(pin "1"
-		)
-		(instances
-			(project "wheelsBoard"
-				(path "/69127114-6359-479f-a1a1-af440f90be3d/daecda86-cddb-4759-b96c-ea8b1b96f1af"
-					(reference "TP6")
-					(unit 1)
-				)
-			)
-			(project "power_Rail"
-				(path "/aa7870c6-fc66-461c-9d29-908d06b1b5db"
-					(reference "TP6")
-					(unit 1)
-				)
-			)
-			(project "SuspensionBoard"
-				(path "/f9dc491a-b8c6-4623-9728-13837ac4bba3/bb9a0353-c4c7-4944-b892-c85c279a5c68"
-					(reference "TP6")
-					(unit 1)
-				)

Commit message: Updated KiCAD Sharepoint
Other:
- moved on the sheet: D12, R30
